File: hardware/UART-RS485_interface-board/UART-RS485_interface-board.kicad_sch (KiCad schematic)
At the start: 19 parts, among them J1 UART (ESP32), J2 3V3, GND, J3 3V3, GND, J8 RS485 (Sensor), U2 MAX3485

Commit message: UART-RS485 Stripboard: Adjust as actually soldered, fixes, add exports
Parts:
- added C2: 10uf, Capacitor_THT:CP_Radial_D8.0mm_P5.00mm, symbol Device:C_Polarized
- added TP6: 3v3, Connector_PinHeader_2.54mm:PinHeader_1x01_P2.54mm_Vertical, symbol Connector:TestPoint
- added TP7: gnd, Connector_PinHeader_2.54mm:PinHeader_1x01_P2.54mm_Vertical, symbol Connector:TestPoint
- C1: footprint Capacitor_THT:C_Disc_D7.0mm_W2.5mm_P5.00mm -> Capacitor_THT:C_Disc_D7.5mm_W5.0mm_P7.50mm
- J1: value UART (ESP32) -> [TX, DIR, RX] UART (ESP32)
- J2, J3: value 3V3, GND -> GND, 3v3
- J8: value RS485 (Sensor) -> [GND, A, B] RS485 (Sensor)
- R35, R37: value 470 -> 3k3
Connections:
- net +3V3: now also C2.1, TP6.1
- net GND: now also C2.2, TP7.1
Other:
- note added: "Note: using MAX485 with 3V3 worked well too but 100mV less voltage swing"
- note added: "RS485 Interface (3V3)"
- note removed: "RS485 Interface"
- title: (none) -> Stripboard UART <=> RS485
